Commit message: removed leading slashes from URDFs

File: packages/duckiebot_interface/urdf/duckiebot.urdf.xacro (robot description, xacro)
@@ -9,17 +9,17 @@
         <!-- START: Duckiebot -->
         <!-- ~/footprint is located at the projection of the wheels axis' center on the ground -->
-        <link name="/${veh}/footprint"/>
+        <link name="${veh}/footprint"/>
         <xacro:if value="${model in ['DB18', 'DB19']}" >
             <!-- START: Duckiebot: DB1X -->
             <xacro:property name="plate_thickness" value="0.003" />
             <!-- /base link is attached to the bottom of the bottom plate -->
-            <link name="/${veh}/base"/>
+            <link name="${veh}/base"/>
             <joint name="${veh}_footprint_to_base" type="fixed">
-                <parent link="/${veh}/footprint" />
-                <child link="/${veh}/base" />
+                <parent link="${veh}/footprint" />
+                <child link="${veh}/base" />
                 <origin xyz="0 0 0.042" />
             </joint>
             <!-- bottom plate -->
-            <link name="/${veh}/bottom_plate">
+            <link name="${veh}/bottom_plate">
                 <visual>
                     <origin xyz="0 0 -${plate_thickness}" />
@@ -30,10 +30,10 @@
             </link>
             <joint name="${veh}_base_to_bottom_plate" type="fixed">
-                <parent link="/${veh}/base" />
-                <child link="/${veh}/bottom_plate" />
+                <parent link="${veh}/base" />
+                <child link="${veh}/bottom_plate" />
                 <origin xyz="0 0 ${plate_thickness}" />
             </joint>
             <!-- top plate -->
-            <link name="/${veh}/top_plate">
+            <link name="${veh}/top_plate">
                 <visual>
                     <origin xyz="0 0 -${plate_thickness}" />
@@ -44,10 +44,10 @@
             </link>
             <joint name="${veh}_bottom_plate_to_top_plate" type="fixed">
-                <parent link="/${veh}/bottom_plate" />
-                <child link="/${veh}/top_plate" />
+                <parent link="${veh}/bottom_plate" />
+                <child link="${veh}/top_plate" />
                 <origin xyz="0 0 0.034" />
             </joint>
             <!-- left motor -->
-            <link name="/${veh}/left_motor">
+            <link name="${veh}/left_motor">
                 <visual>
                     <geometry>
@@ -57,10 +57,10 @@
             </link>
             <joint name="${veh}_base_to_left_motor" type="fixed">
-                <parent link="/${veh}/base" />
-                <child link="/${veh}/left_motor" />
+                <parent link="${veh}/base" />
+                <child link="${veh}/left_motor" />
                 <origin xyz="0 0.023 -0.01" />
             </joint>
             <!-- right motor -->
-            <link name="/${veh}/right_motor">
+            <link name="${veh}/right_motor">
                 <visual>
                     <geometry>
@@ -70,16 +70,16 @@
             </link>
             <joint name="${veh}_base_to_right_motor" type="fixed">
-                <parent link="/${veh}/base" />
-                <child link="/${veh}/right_motor" />
+                <parent link="${veh}/base" />
+                <child link="${veh}/right_motor" />
                 <origin xyz="0 -0.023 -0.01" />
             </joint>
             <!-- left wheel -->
-            <link name="/${veh}/left_wheel_axis"/>
+            <link name="${veh}/left_wheel_axis"/>
             <joint name="${veh}_left_motor_to_left_wheel" type="fixed">
-                <parent link="/${veh}/left_motor" />
-                <child link="/${veh}/left_wheel_axis" />
+                <parent link="${veh}/left_motor" />
+                <child link="${veh}/left_wheel_axis" />
                 <origin xyz="0 0.015 0" />
             </joint>
-            <link name="/${veh}/left_wheel">
+            <link name="${veh}/left_wheel">
                 <visual>
                     <origin rpy="0 0 ${pi}" />
@@ -91,16 +91,16 @@
             <joint name="${veh}_left_wheel_axis_to_left_wheel"
                    type="${'fixed' if model == 'DB18' else 'continuous'}">
-                <parent link="/${veh}/left_wheel_axis" />
-                <child link="/${veh}/left_wheel" />
+                <parent link="${veh}/left_wheel_axis" />
+                <child link="${veh}/left_wheel" />
                 <axis xyz="0 1 0" />
             </joint>
             <!-- right wheel -->
-            <link name="/${veh}/right_wheel_axis"/>
+            <link name="${veh}/right_wheel_axis"/>
             <joint name="${veh}_right_motor_to_right_wheel" type="fixed">
-                <parent link="/${veh}/right_motor" />
-                <child link="/${veh}/right_wheel_axis" />
+                <parent link="${veh}/right_motor" />
+                <child link="${veh}/right_wheel_axis" />
                 <origin xyz="0 -0.015 0" />
             </joint>
-            <link name="/${veh}/right_wheel">
+            <link name="${veh}/right_wheel">
                 <visual>
                     <geometry>
@@ -111,10 +111,10 @@
             <joint name="${veh}_right_wheel_axis_to_right_wheel"
                    type="${'fixed' if model == 'DB18' else 'continuous'}">
-                <parent link="/${veh}/right_wheel_axis" />
-                <child link="/${veh}/right_wheel" />
+                <parent link="${veh}/right_wheel_axis" />
+                <child link="${veh}/right_wheel" />
                 <axis xyz="0 1 0" />
             </joint>
             <!-- caster wheel -->
-            <link name="/${veh}/caster_wheel">
+            <link name="${veh}/caster_wheel">
                 <visual>
                     <geometry>
@@ -124,10 +124,10 @@
             </link>
             <joint name="${veh}_bottom_plate_to_caster_wheel" type="fixed">
-                <parent link="/${veh}/bottom_plate" />
-                <child link="/${veh}/caster_wheel" />
+                <parent link="${veh}/bottom_plate" />
+                <child link="${veh}/caster_wheel" />
                 <origin xyz="-0.083 0 -${plate_thickness}" />
             </joint>
             <!-- front bumper -->
-            <link name="/${veh}/front_bumper">
+            <link name="${veh}/front_bumper">
                 <visual>
                     <geometry>
@@ -137,10 +137,10 @@
             </link>
             <joint name="${veh}_bottom_plate_to_front_bumper" type="fixed">
-                <parent link="/${veh}/bottom_plate" />
-                <child link="/${veh}/front_bumper" />
+                <parent link="${veh}/bottom_plate" />
+                <child link="${veh}/front_bumper" />
                 <origin xyz="0.043 0 0.0155" />
             </joint>
             <!-- back bumper -->
-            <link name="/${veh}/back_bumper">
+            <link name="${veh}/back_bumper">
                 <visual>
                     <geometry>
@@ -150,10 +150,10 @@
             </link>
             <joint name="${veh}_bottom_plate_to_back_bumper" type="fixed">
-                <parent link="/${veh}/bottom_plate" />
-                <child link="/${veh}/back_bumper" />
+                <parent link="${veh}/bottom_plate" />
+                <child link="${veh}/back_bumper" />
                 <origin xyz="-0.1 0 0.0155" rpy="0 0 ${pi}" />
             </joint>
             <!-- camera mount -->
-            <link name="/${veh}/camera_mount">
+            <link name="${veh}/camera_mount">
                 <visual>
                     <geometry>
@@ -163,17 +163,17 @@
             </link>
             <joint name="${veh}_top_plate_to_camera_mount" type="fixed">
-                <parent link="/${veh}/top_plate" />
-                <child link="/${veh}/camera_mount" />
+                <parent link="${veh}/top_plate" />
+                <child link="${veh}/camera_mount" />
                 <origin xyz="0.045 0 0" />
             </joint>
             <!-- camera support -->
-            <link name="/${veh}/camera_support"/>
+            <link name="${veh}/camera_support"/>
             <joint name="${veh}_camera_mount_to_camera_support" type="fixed">
-                <parent link="/${veh}/camera_mount" />
-                <child link="/${veh}/camera_support" />
+                <parent link="${veh}/camera_mount" />
+                <child link="${veh}/camera_support" />
                 <origin xyz="0.01 0 0.023" />
             </joint>
             <!-- camera frame -->
-            <link name="/${veh}/camera_frame">
+            <link name="${veh}/camera_frame">
                 <visual>
                     <geometry>
@@ -184,13 +184,13 @@
             <!-- TODO: this should not be fixed (floating), rotation should be computed from the extrinsics calibration of the camera -->
             <joint name="${veh}_camera_support_to_camera_frame" type="fixed">
-                <parent link="/${veh}/camera_support" />
-                <child link="/${veh}/camera_frame" />
+                <parent link="${veh}/camera_support" />
+                <child link="${veh}/camera_frame" />
                 <origin rpy="0 0.26 0" />
             </joint>
             <!-- camera optical frame -->
-            <link name="/${veh}/camera_optical_frame"/>
+            <link name="${veh}/camera_optical_frame"/>
             <joint name="${veh}_camera_frame_to_camera_optical_frame" type="fixed">
-                <parent link="/${veh}/camera_frame" />
-                <child link="/${veh}/camera_optical_frame" />
+                <parent link="${veh}/camera_frame" />
+                <child link="${veh}/camera_optical_frame" />
                 <origin xyz="0.017 0 0" rpy="-${0.5 * pi} 0 -${0.5 * pi}" />
             </joint>

File: packages/duckiebot_interface/urdf/traffic_light.urdf.xacro (robot description, xacro)
@@ -5,9 +5,9 @@
         <!-- START: Traffic Light -->
         <!-- /footprint is located at the projection of the centroid of the base on the ground -->
-        <link name="/${veh}/footprint"/>
+        <link name="${veh}/footprint"/>
         <!-- TODO: this should not be fixed -->
         <joint name="${veh}_parent_to_footprint" type="fixed">
             <parent link="${parent}" />
-            <child link="/${veh}/footprint" />
+            <child link="${veh}/footprint" />
         </joint>
         <xacro:if value="${model == 'TL19'}" >

File: packages/duckiebot_interface/urdf/watchtower.urdf.xacro (robot description, xacro)
@@ -9,22 +9,22 @@
         <!-- START: Watchtower -->
         <!-- ~/footprint is located at the projection of the centroid of the base on the ground -->
-        <link name="/${veh}/footprint"/>
+        <link name="${veh}/footprint"/>
         <xacro:if value="${model == 'WT18'}" >
             <!-- START: Watchtower: WT18 -->
             <!-- /base link coincides with /footprint -->
-            <link name="/${veh}/base"/>
+            <link name="${veh}/base"/>
             <joint name="${veh}_footprint_to_base" type="fixed">
-                <parent link="/${veh}/footprint" />
-                <child link="/${veh}/base" />
+                <parent link="${veh}/footprint" />
+                <child link="${veh}/base" />
             </joint>
             <!-- camera support -->
-            <link name="/${veh}/camera_support"/>
+            <link name="${veh}/camera_support"/>
             <joint name="${veh}_base_to_camera_support" type="fixed">
-                <parent link="/${veh}/base" />
-                <child link="/${veh}/camera_support" />
+                <parent link="${veh}/base" />
+                <child link="${veh}/camera_support" />
                 <origin xyz="0.08 0.06 0.64" />
             </joint>
             <!-- camera frame -->
-            <link name="/${veh}/camera_frame">
+            <link name="${veh}/camera_frame">
                 <visual>
                     <geometry>
@@ -35,13 +35,13 @@
             <!-- TODO: this should not be fixed (floating), rotation should be computed from the extrinsics calibration of the camera -->
             <joint name="${veh}_camera_support_to_camera_frame" type="fixed">
-                <parent link="/${veh}/camera_support" />
-                <child link="/${veh}/camera_frame" />
+                <parent link="${veh}/camera_support" />
+                <child link="${veh}/camera_frame" />
                 <origin rpy="0 0.26 0" />
             </joint>
             <!-- camera optical frame -->
-            <link name="/${veh}/camera_optical_frame"/>
+            <link name="${veh}/camera_optical_frame"/>
             <joint name="${veh}_camera_frame_to_camera_optical_frame" type="fixed">
-                <parent link="/${veh}/camera_frame" />
-                <child link="/${veh}/camera_optical_frame" />
+                <parent link="${veh}/camera_frame" />
+                <child link="${veh}/camera_optical_frame" />
                 <origin xyz="0.017 0 0" rpy="-${0.5 * pi} 0 -${0.5 * pi}" />
             </joint>

Commit message: added tag_id to duckiebot URDF

File: packages/duckiebot_interface/urdf/duckiebot.urdf.xacro (robot description, xacro)
@@ -5,6 +5,7 @@
         - veh:      Vehicle name (e.g., autobot04)
         - model:    Robot configuration (e.g., DB18)
+        - tag_id:   Robot Tag ID (e.g., 401)
     -->
-    <xacro:macro name="duckiebot" params="veh model">
+    <xacro:macro name="duckiebot" params="veh model tag_id">
         <!-- START: Duckiebot -->
         <!-- ~/footprint is located at the projection of the wheels axis' center on the ground -->
@@ -195,4 +196,13 @@
                 <origin xyz="0.017 0 0" rpy="-${0.5 * pi} 0 -${0.5 * pi}" />
             </joint>
+            <xacro:if value="${tag_id not in ['__NOTSET__']}" >
+                <!-- tag id -->
+                <link name="tag/${tag_id}"/>
+                <joint name="${veh}_top_plate_to_tag_id" type="fixed">
+                    <parent link="${veh}/top_plate" />
+                    <child link="tag/${tag_id}" />
+                    <origin xyz="0.008 0 0.052" />
+                </joint>
+            </xacro:if>
             <!-- END: Duckiebot: DB1X -->
         </xacro:if>
@@ -200,4 +210,4 @@
     </xacro:macro>
     <!--  Spawn Duckiebot  -->
-    <xacro:duckiebot veh="$(arg veh)" model="$(arg model)" />
+    <xacro:duckiebot veh="$(arg veh)" model="$(arg model)" tag_id="$(arg tag_id)" />
 </robot>

Commit message: robot_tag_id and robot_map_name moved to autolab containers

File: packages/duckiebot_interface/urdf/duckiebot.urdf.xacro (robot description, xacro)
@@ -5,7 +5,6 @@
         - veh:      Vehicle name (e.g., autobot04)
         - model:    Robot configuration (e.g., DB18)
-        - tag_id:   Robot Tag ID (e.g., 401)
     -->
-    <xacro:macro name="duckiebot" params="veh model tag_id">
+    <xacro:macro name="duckiebot" params="veh model">
         <!-- START: Duckiebot -->
         <!-- ~/footprint is located at the projection of the wheels axis' center on the ground -->
@@ -196,13 +195,4 @@
                 <origin xyz="0.017 0 0" rpy="-${0.5 * pi} 0 -${0.5 * pi}" />
             </joint>
-            <xacro:if value="${tag_id not in ['__NOTSET__']}" >
-                <!-- tag id -->
-                <link name="tag/${tag_id}"/>
-                <joint name="${veh}_top_plate_to_tag_id" type="fixed">
-                    <parent link="${veh}/top_plate" />
-                    <child link="tag/${tag_id}" />
-                    <origin xyz="0.008 0 0.052" />
-                </joint>
-            </xacro:if>
             <!-- END: Duckiebot: DB1X -->
         </xacro:if>
@@ -210,4 +200,4 @@
     </xacro:macro>
     <!--  Spawn Duckiebot  -->
-    <xacro:duckiebot veh="$(arg veh)" model="$(arg model)" tag_id="$(arg tag_id)" />
+    <xacro:duckiebot veh="$(arg veh)" model="$(arg model)" />
 </robot>

Commit message: added tag_mount to Duckiebot's URDF

File: packages/duckiebot_interface/urdf/duckiebot.urdf.xacro (robot description, xacro)
@@ -8,9 +8,9 @@
     <xacro:macro name="duckiebot" params="veh model">
         <!-- START: Duckiebot -->
-        <!-- ~/footprint is located at the projection of the wheels axis' center on the ground -->
-        <link name="${veh}/footprint"/>
         <xacro:if value="${model in ['DB18', 'DB19']}" >
             <!-- START: Duckiebot: DB1X -->
             <xacro:property name="plate_thickness" value="0.003" />
+            <!-- ~/footprint is located at the projection of the wheels axis' center on the ground -->
+            <link name="${veh}/footprint"/>
             <!-- /base link is attached to the bottom of the bottom plate -->
             <link name="${veh}/base"/>
@@ -153,4 +153,11 @@
                 <child link="${veh}/back_bumper" />
                 <origin xyz="-0.1 0 0.0155" rpy="0 0 ${pi}" />
+            </joint>
+            <!-- tag mount -->
+            <link name="${veh}/tag_mount"/>
+            <joint name="${veh}_top_plate_to_tag_mount" type="fixed">
+                <parent link="${veh}/top_plate" />
+                <child link="${veh}/tag_mount" />
+                <origin xyz="0.008 0 0.051" rpy="${pi} 0 -${0.5 * pi}" />
             </joint>
             <!-- camera mount -->
